File: QUAD_STEP/QUAD_STEP.sch (KiCad schematic (older format))
At the start: 12 parts

Commit message: began H-bridge stage
Parts:
- added C? (x3): 100n, Capacitor_SMD:C_0603_1608Metric, symbol Device:C
- added C?: 10u, Capacitor_SMD:C_0603_1608Metric, symbol Device:C
- added C? (x2): 22p, Capacitor_SMD:C_0402_1005Metric, symbol Device:C
- added C?: 150u 80V, symbol Device:CP
- added C? (x2): 10u, Capacitor_SMD:C_1210_3225Metric_Pad1.42x2.65mm_HandSolder, symbol Device:C
- added J?: ICSP, symbol CUSTOM:ICSP
- added J?: VM, symbol Connector:Conn_01x02_Male
- added Q? (x4): BUK9K45-100E,115, CUSTOM_FP:TRANS_BUK7K12-60EX, symbol CUSTOM:BUK9K45-100E,115
- added R?: 10k, symbol Device:R
- added R? (x2): DNP, symbol Device:R
- added R? (x2): 0R, symbol Device:R
- added U?: ATTINY841-SSU, 14S1, symbol 2019-12-26_17-57-50:ATTINY841-SSU
- added Y?: 10MHz, symbol Device:Crystal
Connections:
- net labels added: 10M_XTAL1, 10M_XTAL2, MCU_MISO, MCU_MOSI, MCU_SCK, MCU_VCC, VCC_IO, VM, ~MCU_RST
- net labels removed: VCC
- wire segments 74 -> 153
Other:
- moved on the sheet: C?, J?, R?, U?

Commit message: finished h bridges, converted to hierarchical layout
Parts:
- removed C?: 22n, Capacitor_SMD:C_0603_1608Metric, symbol Device:C
- removed C? (x2): 2u2, symbol Device:C
- removed C? (x4): 100n, Capacitor_SMD:C_0603_1608Metric, symbol Device:C
- removed C?: 470n, Capacitor_SMD:C_0603_1608Metric, symbol Device:C
- removed C?: 150u 80V, symbol Device:CP
- removed C? (x2): 10u, Capacitor_SMD:C_1210_3225Metric_Pad1.42x2.65mm_HandSolder, symbol Device:C
- removed J?: SPI, symbol Connector:Conn_01x04_Male
- removed J?: AIN, symbol Connector:Conn_01x02_Male
- removed J?: VCC_IO, symbol Connector:Conn_01x02_Male
- removed J?: ENC, symbol Connector:Conn_01x05_Male
- removed J?: VM, symbol Connector:Conn_01x02_Male
- removed Q? (x4): BUK9K45-100E,115, CUSTOM_FP:TRANS_BUK7K12-60EX, symbol CUSTOM:BUK9K45-100E,115
- removed R?: 2R2, symbol Device:R
- removed R? (x2): DNP, symbol Device:R
- removed R? (x2): 0R, symbol Device:R
- removed U?: TMC5160-TA, eTQFP48_9x9, symbol 2019-12-26_03-08-20:TMC5160-TA
- added J? (x4): SCREW TERM, symbol Connector:Conn_01x06_Female
- added J?: USB_B, CUSTOM_FP:CUI_UJ2-BH-W1-TH, symbol Connector:USB_B
- added J?: DB25_Female_MountingHoles, symbol Connector:DB25_Female_MountingHoles
Connections:
- net GND: now also J?.2 (Pin_2), J?.2 (Pin_2), J?.2 (Pin_2), J?.2 (Pin_2)
- new net DRIVE_1/BMA1: J?.3 (Pin_3)
- new net DRIVE_1/BMA2: J?.4 (Pin_4)
- new net DRIVE_1/BMB1: J?.5 (Pin_5)
- new net DRIVE_1/BMB2: J?.6 (Pin_6)
- new net DRIVE_1/VM: J?.1 (Pin_1)
- new net DRIVE_2/BMA1: J?.3 (Pin_3)
- new net DRIVE_2/BMA2: J?.4 (Pin_4)
- new net DRIVE_2/BMB1: J?.5 (Pin_5)
- new net DRIVE_2/BMB2: J?.6 (Pin_6)
- new net DRIVE_2/VM: J?.1 (Pin_1)
- new net DRIVE_3/BMA1: J?.3 (Pin_3)
- new net DRIVE_3/BMA2: J?.4 (Pin_4)
- new net DRIVE_3/BMB1: J?.5 (Pin_5)
- new net DRIVE_3/BMB2: J?.6 (Pin_6)
- new net DRIVE_3/VM: J?.1 (Pin_1)
- new net DRIVE_4/BMA1: J?.3 (Pin_3)
- new net DRIVE_4/BMA2: J?.4 (Pin_4)
- new net DRIVE_4/BMB1: J?.5 (Pin_5)
- new net DRIVE_4/BMB2: J?.6 (Pin_6)
- new net DRIVE_4/VM: J?.1 (Pin_1)
Other:
- note added: "Notes:\nWill need 4x CS lines minimum; 4X DRV_ENN would be nice. Logical OR for DIAG ports? This would combine 8 into 1, with no additional components (Open collector output)\nAlmost no point in providing step/dir from MCU, as this can be handled through driver serial interface\nMove away from ATTINY. For pennies more, you can break out everything."

Commit message: added more components, fleshed out DB-25 interface, added PSoC
Parts:
- added J? (x4): SCREW TERM, symbol Connector:Conn_01x05_Female
- added J?: SCREW_TERM, symbol Connector:Conn_01x02_Female
- added J?: SPARE_IN, symbol Connector:Conn_01x05_Female
- added J?: SPARE_OUT, symbol Connector:Conn_01x03_Female
- added R? (x75): 0R, symbol Device:R
- added U?: CY8C5468AXI-LP106, TQFP-100, symbol 2019-12-30_03-28-16:CY8C5468AXI-LP106
- J?: footprint (none) -> Connector_PinHeader_2.54mm:PinHeader_2x03_P2.54mm_Vertical
Connections:
- net DRIVE_1/CS: now also R?.1, R?.1
- net DRIVE_1/DIAG0: now also R?.2
- net DRIVE_1/DIAG1: now also R?.2
- net DRIVE_1/ENC_A: now also J?.5 (Pin_5)
- net DRIVE_1/ENC_B: now also J?.4 (Pin_4)
- net DRIVE_1/ENC_N: now also J?.3 (Pin_3)
- net DRIVE_1/MISO: now also R?.1, R?.1
- net DRIVE_1/MOSI: now also R?.1, R?.1
- net DRIVE_1/REFL_STEP: now also R?.1, R?.1
- net DRIVE_1/REFR_DIR: now also R?.1, R?.1
- net DRIVE_1/SCK: now also R?.1, R?.1
- net DRIVE_1/VCC_IO: now also R?.1
- net DRIVE_2/CS: now also R?.1, R?.1
- net DRIVE_2/ENC_A: now also J?.5 (Pin_5)
- net DRIVE_2/ENC_B: now also J?.4 (Pin_4)
- net DRIVE_2/ENC_N: now also J?.3 (Pin_3)
- net DRIVE_2/MISO: now also R?.1, R?.1
- net DRIVE_2/MOSI: now also R?.1, R?.1
- net DRIVE_2/REFL_STEP: now also R?.1, R?.1
- net DRIVE_2/REFR_DIR: now also R?.1, R?.1
- net DRIVE_2/SCK: now also R?.1, R?.1
- net DRIVE_2/VCC_IO: now also R?.1
- net DRIVE_3/CS: now also R?.1, R?.1
- net DRIVE_3/ENC_A: now also J?.5 (Pin_5)
- net DRIVE_3/ENC_B: now also J?.4 (Pin_4)
- net DRIVE_3/ENC_N: now also J?.3 (Pin_3)
- net DRIVE_3/MISO: now also R?.1, R?.1
- net DRIVE_3/MOSI: now also R?.1, R?.1
- net DRIVE_3/REFL_STEP: now also R?.1, R?.1
- net DRIVE_3/REFR_DIR: now also R?.1, R?.1
- net DRIVE_3/SCK: now also R?.1, R?.1
- net DRIVE_3/VCC_IO: now also R?.1
- net DRIVE_4/CS: now also R?.1, R?.1
- net DRIVE_4/ENC_A: now also J?.5 (Pin_5)
- net DRIVE_4/ENC_B: now also J?.4 (Pin_4)
- net DRIVE_4/ENC_N: now also J?.3 (Pin_3)
- net DRIVE_4/MISO: now also R?.1, R?.1
- net DRIVE_4/MOSI: now also R?.1, R?.1
- net DRIVE_4/REFL_STEP: now also R?.1, R?.1
- net DRIVE_4/REFR_DIR: now also R?.1, R?.1
- net DRIVE_4/SCK: now also R?.1, R?.1
- net DRIVE_4/VCC_IO: now also R?.1
- net GND: now also J?.0 (PAD), J?.18 (P18), J?.19 (P19), J?.20 (P20), J?.21 (P21), J?.22 (P22), J?.23 (P23), J?.24 (P24), J?.25 (P25), J?.4 (GND), J?.5 (Shield), J?.1 (Pin_1), J?.1 (Pin_1), J?.1 (Pin_1), J?.1 (Pin_1), J?.1 (Pin_1)
- net at U?.10 (PA3): now also R?.2
- net at U?.11 (PA2): now also R?.2
- net at U?.12 (PA1): now also R?.2
- net at U?.13 (PA0): now also R?.2
- net ~ATM_ENA: now reaches U?.5 (PB2)
- net ~ATM_ENA: now also R?.2, R?.2, R?.2, R?.2
- net VCC_CONT: now reaches J?.1 (VBUS)
- net VCC_CONT: now also J?.2, R?.1, J?.2 (Pin_2), R?.1, R?.1, R?.1, R?.1, R?.2, R?.2, R?.2, R?.2, R?.2
- net ~PAR_ENA: now reaches J?.1
- net ~PAR_ENA: now also R?.2, R?.2, R?.2, R?.2
- net at J?.10: now also J?.4 (Pin_4)
- net at J?.11: now also J?.3 (Pin_3)
- net at J?.12: now also J?.2 (Pin_2)
- net at J?.13: now also J?.1 (Pin_1)
- net at J?.14 (P14): now also J?.3 (Pin_3)
- net at J?.15 (P15): now also J?.5 (Pin_5)
- net at J?.16 (P16): now also J?.2 (Pin_2)
- net at J?.17 (P17): now also J?.1 (Pin_1)
- net PAR_STEP1: now reaches J?.2
- net PAR_STEP1: now also R?.2
- net PAR_DIR1: now reaches J?.3
- net PAR_DIR1: now also R?.2
- net PAR_STEP2: now reaches J?.4
- net PAR_STEP2: now also R?.2
- net PAR_DIR2: now reaches J?.5
- net PAR_DIR2: now also R?.2
- net PAR_STEP3: now reaches J?.6
- net PAR_STEP3: now also R?.2
- net PAR_DIR3: now reaches J?.7
- net PAR_DIR3: now also R?.2
- net PAR_STEP4: now reaches J?.8
- net PAR_STEP4: now also R?.2
- net PAR_DIR4: now reaches J?.9
- net PAR_DIR4: now also R?.2
- net MCU_MISO renamed ATM_MISO
- net ATM_MISO: now also R?.2, R?.2, R?.2, R?.2
- net MCU_MOSI renamed ATM_MOSI
- net ATM_MOSI: now also R?.2, R?.2, R?.2, R?.2
- net MCU_SCK renamed ATM_SCK
- net ATM_SCK: now also R?.2, R?.2, R?.2, R?.2
- net MCU_VCC: no longer names the net of C?.1, C?.1, U?.1 (VCC)
- net MCU_VCC: now also R?.1; no longer J?.2, R?.1
- net ~MCU_RST renamed ~ATM_RST
- new net: J?.2 (Pin_2), R?.2 (x4)
- new net ATM_CS1: R?.1, R?.2
- new net ATM_CS2: R?.1, R?.2
- new net ATM_CS3: R?.1, R?.2
- new net ATM_CS4: R?.1, R?.2
- new net CYP_CS1: R?.2
- new net CYP_CS2: R?.2
- new net CYP_CS3: R?.2
- new net CYP_CS4: R?.2
- new net CYP_DIR1: R?.2
- new net CYP_DIR2: R?.2
- new net CYP_DIR3: R?.2
- new net CYP_DIR4: R?.2
- new net CYP_MISO: R?.2, R?.2, R?.2, R?.2
- new net CYP_MOSI: R?.2, R?.2, R?.2, R?.2
- new net CYP_SCK: R?.2, R?.2, R?.2, R?.2
- new net CYP_STEP1: R?.2
- new net CYP_STEP2: R?.2
- new net CYP_STEP3: R?.2
- new net CYP_STEP4: R?.2
- new net DIAG_0_1: R?.1
- new net DIAG_1_1: R?.1
- new net DRIVE_1/~DRV_ENN: R?.1, R?.1, R?.1
- new net DRIVE_2/~DRV_ENN: R?.1, R?.1, R?.1
- new net DRIVE_3/~DRV_ENN: R?.1, R?.1, R?.1
- new net DRIVE_4/~DRV_ENN: R?.1, R?.1, R?.1
- new net ~CYP_ENA_1: R?.2
- new net ~CYP_ENA_2: R?.2
- new net ~CYP_ENA_3: R?.2
- new net ~CYP_ENA_4: R?.2
Other:
- note added: "Notes:\n3x SPI\n4x CS lines minimum\n4X DRV_ENN\n8x DIAG ports (consider using I2C I/O expander such as TCA9554DBR. This has interrupt output capabilities. 2x for I2C, 1x for interrupt)\n4x STEP\n4x DIR\n\n22 total\n\n\nATMEGA 32u4\nhttps://www.digikey.com/product-detail/en/microchip-technology/ATMEGA32U4RC-AU/ATMEGA32U4RC-AU-ND/2507982\n\nPSoC 4 may be a much better/cheaper alternative. https://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"
- note removed: "Notes:\nWill need 4x CS lines minimum; 4X DRV_ENN would be nice. Logical OR for DIAG ports? This would combine 8 into 1, with no additional components (Open collector output)\nAlmost no point in providing step/dir from MCU, as this can be handled through driver serial interface\nMove away from ATTINY. For pennies more, you can break out everything."
- moved on the sheet: J?
