File: QUAD_STEP/QUAD_STEP.sch (KiCad schematic (older format))
At the start: 130 parts, among them J1 DB25_Female_LCNC, J10 ENC_HEADER, J11 ENC_HEADER, J12 PSoC_PROG, J13 POWER, J14 SCREW TERM, J15 SCREW TERM, J16 ENC_HEADER, J17 ENC_HEADER, J18 SCREW TERM, J19 SCREW TERM, J2 SCREW_TERM, J20 CYP_I2C, J21 CLK16, J22 CLK16, J23 CLK16, J24 CLK16, J3 USB_B, J4 SPARE_IN, J5 SPARE_OUT, J6 PROG_V, J7 RUN_V, J8 ICSP, J9 GPIO_header, U1 ATTINY841-SSU, U2 CY8C5468AXI-LP106, Y1 10MHz

Commit message: beginning layout
Parts:
- removed J21, J22, J23, J24: CLK16, symbol Connector:Conn_01x01_Male
- removed J3: USB_B, CUSTOM_FP:CUI_UJ2-BH-W1-TH, symbol Connector:USB_B
- removed R10, R11, R12, R13, R14, R15, R16, R17, R26, R27, R28, R32, R33, R34, R35, R40, R42, R44, R45: 0R, symbol Device:R
- added F1, F2, F3, F4: BLADE_Fuse, CUSTOM:keystone_3549_2_fuseholder_THT, symbol CUSTOM:BLADE_Fuse
- added J3: USB_B, CUSTOM:CUI_UJ2-BH-W1-TH, symbol CUSTOM:USB_B
- added JP1, JP10, JP11, JP12, JP13, JP14, JP15, JP16, JP17, JP18, JP19, JP2, JP3, JP4, JP5, JP6, JP7, JP8, JP9: SolderJumper_2_Open, CUSTOM:small_triangle_jumper, symbol Jumper:SolderJumper_2_Open
- added TP1, TP2, TP3, TP4: CLK16, TestPoint:TestPoint_Pad_D1.0mm, symbol Connector:TestPoint
- J1: footprint (none) -> Connector_Dsub:DSUB-25_Female_Horizontal_P2.77x2.84mm_EdgePinOffset7.70mm_Housed_MountingHolesOffset9.12mm
- J14, J15, J18, J19: footprint (none) -> CUSTOM:CUI_TB002-500-06BE
- J2: footprint (none) -> CUSTOM:PHOENIX_1935161
- R1, R162, R163, R18, R19, R2, R20, R21, R22, R23, R24, R25, R29, R3, R30, R31, R36, R37, R38, R39, R4, R41, R43, R46, R47, R48, R49, R5, R50, R51, R52, R53, R54, R55, R56, R57, R58, R59, R6, R60, R61, R62, R63, R64, R65, R66, R67, R68, R69, R7, R70, R71, R72, R73, R74, R75, R76, R77, R78, R79, R8, R80, R81, R82, R83, R84, R85, R9: footprint (none) -> Resistor_SMD:R_0603_1608Metric_Pad1.05x0.95mm_HandSolder
- U1: footprint 14S1 -> CUSTOM:ATTINY841-SSU
- U2: footprint TQFP-100 -> CUSTOM:CY8C5468AXI-LP106
- Y1: footprint (none) -> Crystal:Crystal_SMD_HC49-SD_HandSoldering
Connections:
- net ATM_CS1: now also JP4.1 (A)
- net ATM_MISO: now also JP8.1 (A)
- net ATM_MOSI: now also JP6.1 (A)
- net ATM_SCK: now also JP2.1 (A)
- net CYP_CS1: now also JP3.1 (A)
- net CYP_DIR1: now also JP14.1 (A)
- net CYP_MISO: now also JP7.1 (A)
- net CYP_MOSI: now also JP5.1 (A)
- net CYP_SCK: now also JP1.1 (A)
- net CYP_STEP1: now also JP12.1 (A)
- net DIAG_0_1: now also JP18.2 (B)
- net DIAG_1_1: now also JP19.2 (B)
- net DRIVE_1/CLK16: now also TP1.1
- net DRIVE_1/CS: now also JP3.2 (B), JP4.2 (B)
- net DRIVE_1/DIAG0: now also JP18.1 (A)
- net DRIVE_1/DIAG1: now also JP19.1 (A)
- net DRIVE_1/MISO: now also JP7.2 (B), JP8.2 (B)
- net DRIVE_1/MOSI: now also JP5.2 (B), JP6.2 (B)
- net DRIVE_1/REFL_STEP: now also JP12.2 (B), JP13.2 (B)
- net DRIVE_1/REFR_DIR: now also JP14.2 (B), JP15.2 (B)
- net DRIVE_1/SCK: now also JP1.2 (B), JP2.2 (B)
- net DRIVE_1/VCC_IO: now also JP16.2 (B)
- net DRIVE_1/VM: now also F1.1, F1.2; no longer J14.1 (Pin_1)
- net DRIVE_1/~DRV_ENN: now also JP10.2 (B), JP11.2 (B), JP9.2 (B)
- net DRIVE_2/CLK16: now also TP2.1
- net DRIVE_2/VM: now also F2.1, F2.2; no longer J15.1 (Pin_1)
- net DRIVE_3/CLK16: now also TP3.1
- net DRIVE_3/VM: now also F3.1, F3.2; no longer J18.1 (Pin_1)
- net DRIVE_4/CLK16: now also TP4.1
- net DRIVE_4/VM: now also F4.1, F4.2; no longer J19.1 (Pin_1)
- net GND: now also J3.4 (GND), J3.SH1, J3.SH2
- net PAR_DIR1: now also JP15.1 (A)
- net PAR_STEP1: now also JP13.1 (A)
- net USBIO_D+: now also J3.3 (D+)
- net USBIO_D-: now also J3.2 (D-)
- net VCC_CONT: now also J3.1 (VBUS), JP16.1 (A), JP17.2 (B)
- net ~ATM_ENA: now also JP10.1 (A)
- net ~CYP_ENA_1: now also JP9.1 (A)
- net ~PAR_ENA: now also JP11.1 (A)
- net at J10.2 (Pin_2): now also JP17.1 (A)
- new net: F1.3, F1.4, J14.1 (Pin_1)
- new net: F2.3, F2.4, J15.1 (Pin_1)
- new net: F4.3, F4.4, J19.1 (Pin_1)
- new net: F3.3, F3.4, J18.1 (Pin_1)

Commit message: complebegan adding 3D files
Parts:
- removed R164: DNP, Resistor_SMD:R_0603_1608Metric_Pad1.05x0.95mm_HandSolder, symbol Device:R
- removed R18, R19, R20, R21, R22, R23, R24, R25, R29, R30, R31, R36, R37, R38, R39, R41, R43, R46, R47, R48, R49, R50, R51, R52, R53, R54, R55, R56, R57, R58, R59, R60, R61, R62, R63, R64, R65, R66, R67, R68, R69, R70, R71, R72, R73, R74, R75, R76, R77, R78, R79, R80, R81, R82, R83, R84, R85: 0R, Resistor_SMD:R_0603_1608Metric_Pad1.05x0.95mm_HandSolder, symbol Device:R
- added JP20, JP21, JP22, JP23, JP24, JP25, JP26, JP27, JP28, JP29, JP30, JP31, JP32, JP33, JP34, JP35, JP36, JP37, JP38, JP39, JP40, JP41, JP42, JP43, JP44, JP45, JP46, JP47, JP48, JP49, JP50, JP51, JP52, JP53, JP54, JP55, JP56, JP57, JP58, JP59, JP60, JP61, JP62, JP63, JP64, JP65, JP66, JP67, JP68, JP69, JP70, JP71, JP72, JP73, JP74, JP75, JP76: SolderJumper_2_Open, CUSTOM:small_triangle_jumper, symbol Jumper:SolderJumper_2_Open
- added TP5: ATM_SPARE, TestPoint:TestPoint_Pad_D1.0mm, symbol Connector:TestPoint
- Y1: footprint Crystal:Crystal_SMD_HC49-SD_HandSoldering -> CUSTOM:CX5032GB10000H0PESZZ; DPN 631-1011-1-ND -> 478-4358-1-ND; MPN FC4SDCBMF10.0-T1 -> CX5032GB10000H0PESZZ
Connections:
- net ATM_CS2: now also JP23.1 (A)
- net ATM_CS3: now also JP42.1 (A)
- net ATM_CS4: now also JP50.1 (A)
- net ATM_MISO: now also JP27.1 (A), JP46.1 (A), JP54.1 (A)
- net ATM_MOSI: now also JP25.1 (A), JP44.1 (A), JP52.1 (A)
- net ATM_SCK: now also JP21.1 (A), JP40.1 (A), JP48.1 (A)
- net CYP_CS2: now also JP22.1 (A)
- net CYP_CS3: now also JP41.1 (A)
- net CYP_CS4: now also JP49.1 (A)
- net CYP_DIR2: now also JP33.1 (A)
- net CYP_DIR3: now also JP63.1 (A)
- net CYP_DIR4: now also JP67.1 (A)
- net CYP_MISO: now also JP26.1 (A), JP45.1 (A), JP53.1 (A)
- net CYP_MOSI: now also JP24.1 (A), JP43.1 (A), JP51.1 (A)
- net CYP_SCK: now also JP20.1 (A), JP39.1 (A), JP47.1 (A)
- net CYP_STEP2: now also JP31.1 (A)
- net CYP_STEP3: now also JP61.1 (A)
- net CYP_STEP4: now also JP65.1 (A)
- net DIAG_0_2: now also JP37.2 (B)
- net DIAG_0_3: now also JP73.2 (B)
- net DIAG_0_4: now also JP75.2 (B)
- net DIAG_1_2: now also JP38.2 (B)
- net DIAG_1_3: now also JP74.2 (B)
- net DIAG_1_4: now also JP76.2 (B)
- net DRIVE_1/ENC_A: now also J10.4 (Pin_4); no longer J10.5 (Pin_5)
- net DRIVE_1/ENC_B: now also J10.5 (Pin_5); no longer J10.4 (Pin_4)
- net DRIVE_2/CS: now also JP22.2 (B), JP23.2 (B)
- net DRIVE_2/DIAG0: now also JP37.1 (A)
- net DRIVE_2/DIAG1: now also JP38.1 (A)
- net DRIVE_2/MISO: now also JP26.2 (B), JP27.2 (B)
- net DRIVE_2/MOSI: now also JP24.2 (B), JP25.2 (B)
- net DRIVE_2/REFL_STEP: now also JP31.2 (B), JP32.2 (B)
- net DRIVE_2/REFR_DIR: now also JP33.2 (B), JP34.2 (B)
- net DRIVE_2/SCK: now also JP20.2 (B), JP21.2 (B)
- net DRIVE_2/VCC_IO: now also JP35.2 (B)
- net DRIVE_2/~DRV_ENN: now also JP28.2 (B), JP29.2 (B), JP30.2 (B)
- net DRIVE_3/CS: now also JP41.2 (B), JP42.2 (B)
- net DRIVE_3/DIAG0: now also JP73.1 (A)
- net DRIVE_3/DIAG1: now also JP74.1 (A)
- net DRIVE_3/MISO: now also JP45.2 (B), JP46.2 (B)
- net DRIVE_3/MOSI: now also JP43.2 (B), JP44.2 (B)
- net DRIVE_3/REFL_STEP: now also JP61.2 (B), JP62.2 (B)
- net DRIVE_3/REFR_DIR: now also JP63.2 (B), JP64.2 (B)
- net DRIVE_3/SCK: now also JP39.2 (B), JP40.2 (B)
- net DRIVE_3/VCC_IO: now also JP69.2 (B)
- net DRIVE_3/~DRV_ENN: now also JP55.2 (B), JP56.2 (B), JP57.2 (B)
- net DRIVE_4/CS: now also JP49.2 (B), JP50.2 (B)
- net DRIVE_4/DIAG0: now also JP75.1 (A)
- net DRIVE_4/DIAG1: now also JP76.1 (A)
- net DRIVE_4/MISO: now also JP53.2 (B), JP54.2 (B)
- net DRIVE_4/MOSI: now also JP51.2 (B), JP52.2 (B)
- net DRIVE_4/REFL_STEP: now also JP65.2 (B), JP66.2 (B)
- net DRIVE_4/REFR_DIR: now also JP67.2 (B), JP68.2 (B)
- net DRIVE_4/SCK: now also JP47.2 (B), JP48.2 (B)
- net DRIVE_4/VCC_IO: now also JP70.2 (B)
- net DRIVE_4/~DRV_ENN: now also JP58.2 (B), JP59.2 (B), JP60.2 (B)
- net PAR_DIR2: now also JP34.1 (A)
- net PAR_DIR3: now also JP64.1 (A)
- net PAR_DIR4: now also JP68.1 (A)
- net PAR_STEP2: now also JP32.1 (A)
- net PAR_STEP3: now also JP62.1 (A)
- net PAR_STEP4: now also JP66.1 (A)
- net VCC_CONT: now also JP35.1 (A), JP36.2 (B), JP69.1 (A), JP70.1 (A), JP71.2 (B), JP72.2 (B)
- net ~ATM_ENA: now also JP29.1 (A), JP56.1 (A), JP59.1 (A)
- net ~CYP_ENA_2: now also JP28.1 (A)
- net ~CYP_ENA_3: now also JP55.1 (A)
- net ~CYP_ENA_4: now also JP58.1 (A)
- net ~PAR_ENA: now also JP30.1 (A), JP57.1 (A), JP60.1 (A)
- net at U1.6 (PA7): now also TP5.1
- net at J11.2 (Pin_2): now also JP36.1 (A)
- net at J17.2 (Pin_2): now also JP72.1 (A)
- net at J16.2 (Pin_2): now also JP71.1 (A)
- no-connect marks 31 -> 30
Other:
- moved on the sheet: C1, C2, R1

Commit message: changed scope to 5 axis, preliminary completion of component positioning
Parts:
- removed J13: POWER, Connector_PinHeader_2.54mm:PinHeader_1x06_P2.54mm_Vertical, symbol Connector:Conn_01x06_Male
- removed J5: SPARE_OUT, Connector_PinHeader_2.54mm:PinHeader_1x03_P2.54mm_Vertical, symbol Connector:Conn_01x03_Female
- removed J6: PROG_V, Connector_PinHeader_2.54mm:PinHeader_1x02_P2.54mm_Vertical, symbol Connector:Conn_01x02_Male
- removed J7: RUN_V, Connector_PinHeader_2.54mm:PinHeader_1x02_P2.54mm_Vertical, symbol Connector:Conn_01x02_Male
- removed J9: GPIO_header, Connector_PinHeader_2.54mm:PinHeader_1x10_P2.54mm_Vertical, symbol Connector:Conn_01x10_Male
- removed R1, R2, R3, R4, R6, R7, R8, R9: 0R, Resistor_SMD:R_0603_1608Metric_Pad1.05x0.95mm_HandSolder, symbol Device:R
- added F5: BLADE_Fuse, CUSTOM_FP:keystone_3549_2_fuseholder_THT, symbol CUSTOM:BLADE_Fuse
- added H1, H2, H3, H4: MountingHole_Pad, MountingHole:MountingHole_4.5mm_Pad_Via, symbol Mechanical:MountingHole_Pad
- added J5: ENC_HEADER, Connector_PinHeader_2.54mm:PinHeader_1x05_P2.54mm_Vertical, symbol Connector:Conn_01x05_Female
- added J6: Conn_02x02_Odd_Even, Connector_PinHeader_2.54mm:PinHeader_2x02_P2.54mm_Vertical, symbol Connector_Generic:Conn_02x02_Odd_Even
- added J7: CYP_GPIO, Connector_PinHeader_2.54mm:PinHeader_2x05_P2.54mm_Vertical, symbol Connector_Generic:Conn_02x05_Odd_Even
- added J9: SCREW TERM, CUSTOM_FP:CUI_TB002-500-06BE, symbol Connector:Conn_01x06_Female
- added JP77, JP78, JP79, JP80, JP81, JP82, JP83, JP84, JP85, JP86, JP87, JP88, JP89, JP90, JP91, JP92, JP93, JP94, JP95, JP96, JP97, JP98, JP99: SolderJumper_2_Open, CUSTOM_FP:small_triangle_jumper, symbol Jumper:SolderJumper_2_Open
- added TP6: CLK16, TestPoint:TestPoint_Pad_D1.0mm, symbol Connector:TestPoint
- C5, C7: value 22p -> 18p; footprint Capacitor_SMD:C_0402_1005Metric -> Capacitor_SMD:C_0603_1608Metric_Pad1.05x0.95mm_HandSolder; DPN 587-5869-1-ND -> 399-17581-1-ND; MPN C0402C220K4RAC7867 -> C0603C180K5RACAUTO
- J2: value SCREW_TERM -> MTA-100; footprint CUSTOM:PHOENIX_1935161 -> CUSTOM_FP:640456-2; DPN 277-1667-ND -> A1921-ND; MPN 1935161 -> 640456-2
- TP5: value ATM_SPARE -> PAR_SPARE
Connections:
- net ATM_CS1: now also U1.13 (PA0)
- net ATM_CS2: now also U1.12 (PA1)
- net ATM_CS3: now also U1.11 (PA2)
- net ATM_CS4: now also U1.10 (PA3)
- net ATM_MISO: now also JP87.1 (A)
- net ATM_MOSI: now also JP85.1 (A)
- net ATM_SCK: now also JP81.1 (A)
- net CYP_MISO: now also JP86.1 (A)
- net CYP_MOSI: now also JP84.1 (A)
- net CYP_SCK: now also JP80.1 (A)
- net DRIVE_2/ENC_A: now also J11.4 (Pin_4); no longer J11.5 (Pin_5)
- net DRIVE_2/ENC_B: now also J11.5 (Pin_5); no longer J11.4 (Pin_4)
- net DRIVE_3/ENC_A: now also J16.4 (Pin_4); no longer J16.5 (Pin_5)
- net DRIVE_3/ENC_B: now also J16.5 (Pin_5); no longer J16.4 (Pin_4)
- net DRIVE_4/ENC_A: now also J17.4 (Pin_4); no longer J17.5 (Pin_5)
- net DRIVE_4/ENC_B: now also J17.5 (Pin_5); no longer J17.4 (Pin_4)
- net GND: now also J12.5 (Pin_5), H1.1, H2.1, H3.1, H4.1, J5.1 (Pin_1), J9.2 (Pin_2); no longer J12.4 (Pin_4)
- net SWDCLK: now also J12.1 (Pin_1); no longer J12.2 (Pin_2)
- net SWDIO: now also J12.2 (Pin_2); no longer J12.1 (Pin_1)
- net VCCD: now also JP77.2 (B)
- net VCC_CONT: now also J6.3 (Pin_3), JP95.1 (A), JP96.2 (B), JP99.1 (A)
- net VDDA: now also JP78.2 (B)
- net VDDD: now also JP79.2 (B)
- net VTARG: now also J12.4 (Pin_4), J6.1 (Pin_1); no longer J12.5 (Pin_5)
- net ~ATM_ENA: now also JP89.1 (A)
- net ~PAR_ENA: now also JP90.1 (A)
- net at C1.1, C2.1, U1.1 (VCC): now also JP99.2 (B)
- net at TP5.1: now also J1.17 (P17); no longer U1.6 (PA7)
- net PAR_STEP5: now reaches J1.14 (P14)
- net PAR_STEP5: now also JP92.1 (A)
- net PAR_DIR5: now reaches J1.16 (P16)
- net PAR_DIR5: now also JP94.1 (A)
- net at U2.22 (P12): now also J7.1 (Pin_1)
- net at U2.23 (P13): now also J7.2 (Pin_2)
- net at U2.24 (P14): now also J7.3 (Pin_3)
- net at U2.25 (P15): now also J7.4 (Pin_4)
- net at U2.27 (P16): now also J7.5 (Pin_5)
- net at U2.28 (P17): now also J7.6 (Pin_6)
- net at U2.31 (P54): now also J7.7 (Pin_7)
- net at U2.32 (P55): now also J7.8 (Pin_8)
- net at U2.33 (P56): now also J7.9 (Pin_9)
- net at U2.34 (P57): now also J7.10 (Pin_10)
- net DIAG_1_5: now reaches U2.44 (P30)
- net DIAG_1_5: now also JP98.2 (B)
- net DIAG_0_5: now reaches U2.45 (P31)
- net DIAG_0_5: now also JP97.2 (B)
- net CYP_DIR5: now reaches U2.46 (P32)
- net CYP_DIR5: now also JP93.1 (A)
- net CYP_STEP5: now reaches U2.47 (P33)
- net CYP_STEP5: now also JP91.1 (A)
- net ~CYP_ENA_5: now reaches U2.48 (P34)
- net ~CYP_ENA_5: now also JP88.1 (A)
- net CYP_CS5: now reaches U2.95 (P20)
- net CYP_CS5: now also JP82.1 (A)
- new net: J6.2 (Pin_2), J6.4 (Pin_4), JP77.1 (A), JP78.1 (A), JP79.1 (A)
- new net: F5.3, F5.4, J9.1 (Pin_1)
- new net: J5.2 (Pin_2), JP96.1 (A)
- new net ATM_CS5: JP83.1 (A), U1.6 (PA7)
- new net DRIVE_5/BMA1: J9.3 (Pin_3)
- new net DRIVE_5/BMA2: J9.4 (Pin_4)
- new net DRIVE_5/BMB1: J9.5 (Pin_5)
- new net DRIVE_5/BMB2: J9.6 (Pin_6)
- new net DRIVE_5/CLK16: TP6.1
- new net DRIVE_5/CS: JP82.2 (B), JP83.2 (B)
- new net DRIVE_5/DIAG0: JP97.1 (A)
- new net DRIVE_5/DIAG1: JP98.1 (A)
- new net DRIVE_5/ENC_A: J5.4 (Pin_4)
- new net DRIVE_5/ENC_B: J5.5 (Pin_5)
- new net DRIVE_5/ENC_N: J5.3 (Pin_3)
- new net DRIVE_5/MISO: JP86.2 (B), JP87.2 (B)
- new net DRIVE_5/MOSI: JP84.2 (B), JP85.2 (B)
- new net DRIVE_5/REFL_STEP: JP91.2 (B), JP92.2 (B)
- new net DRIVE_5/REFR_DIR: JP93.2 (B), JP94.2 (B)
- new net DRIVE_5/SCK: JP80.2 (B), JP81.2 (B)
- new net DRIVE_5/VCC_IO: JP95.2 (B)
- new net DRIVE_5/VM: F5.1, F5.2
- new net DRIVE_5/~DRV_ENN: JP88.2 (B), JP89.2 (B), JP90.2 (B)
- no-connect marks 30 -> 24
