File: QUAD_STEP/QUAD_STEP.kicad_pcb (KiCad board)
At the start: 4 copper layers, 100 x 100 mm, 298 parts, among them J1 DB25_Female_LCNC, J10 ENC_HEADER, J11 ENC_HEADER, J12 PSoC_PROG, J13 POWER, J14 SCREW TERM, J15 SCREW TERM, J16 ENC_HEADER, J17 ENC_HEADER, J18 SCREW TERM, J19 SCREW TERM, J2 SCREW_TERM, J20 CYP_I2C, J3 USB_B, J4 SPARE_IN, J5 SPARE_OUT, J6 PROG_V, J7 RUN_V, J8 ICSP, J9 GPIO_header, Q1 BUK9K45-100E,115, Q10 BUK9K45-100E,115, Q11 BUK9K45-100E,115, Q12 BUK9K45-100E,115, Q13 BUK9K45-100E,115, Q14 BUK9K45-100E,115, Q15 BUK9K45-100E,115, Q16 BUK9K45-100E,115, Q2 BUK9K45-100E,115, Q3 BUK9K45-100E,115, Q4 BUK9K45-100E,115, Q5 BUK9K45-100E,115, Q6 BUK9K45-100E,115, Q7 BUK9K45-100E,115, Q8 BUK9K45-100E,115, Q9 BUK9K45-100E,115, U1 ATTINY841-SSU, U2 CY8C5468AXI-LP106, U3 TMC5160-TA, U4 TMC5160-TA, U5 TMC5160-TA, U6 TMC5160-TA, Y1 10MHz

Commit message: complebegan adding 3D files
Parts:
- removed R164: DNP, Resistor_SMD:R_0603_1608Metric_Pad1.05x0.95mm_HandSolder
- removed R18, R19, R20, R21, R22, R23, R24, R25, R29, R30, R31, R36, R37, R38, R39, R41, R43, R46, R47, R48, R49, R50, R51, R52, R53, R54, R55, R56, R57, R58, R59, R60, R61, R62, R63, R64, R65, R66, R67, R68, R69, R70, R71, R72, R73, R74, R75, R76, R77, R78, R79, R80, R81, R82, R83, R84, R85: 0R, Resistor_SMD:R_0603_1608Metric_Pad1.05x0.95mm_HandSolder
- added JP20: SolderJumper_2_Open, CUSTOM:small_triangle_jumper, F.Cu at (10.2, -130.8)
- added JP21: SolderJumper_2_Open, CUSTOM:small_triangle_jumper, B.Cu at (10.2, -130.8)
- added JP22: SolderJumper_2_Open, CUSTOM:small_triangle_jumper, F.Cu at (10.2, -128.3)
- added JP23: SolderJumper_2_Open, CUSTOM:small_triangle_jumper, B.Cu at (10.2, -128.3)
- added JP24: SolderJumper_2_Open, CUSTOM:small_triangle_jumper, F.Cu at (10.2, -125.7)
- added JP25: SolderJumper_2_Open, CUSTOM:small_triangle_jumper, B.Cu at (10.2, -125.7)
- added JP26: SolderJumper_2_Open, CUSTOM:small_triangle_jumper, F.Cu at (10.2, -123.2)
- added JP27: SolderJumper_2_Open, CUSTOM:small_triangle_jumper, B.Cu at (10.2, -123.2)
- added JP28: SolderJumper_2_Open, CUSTOM:small_triangle_jumper, F.Cu at (10.2, -120.7)
- added JP29: SolderJumper_2_Open, CUSTOM:small_triangle_jumper, B.Cu at (10.2, -120.7)
- added JP30: SolderJumper_2_Open, CUSTOM:small_triangle_jumper, F.Cu at (10.2, -118.1)
- added JP31: SolderJumper_2_Open, CUSTOM:small_triangle_jumper, F.Cu at (10.2, -115.6)
- added JP32: SolderJumper_2_Open, CUSTOM:small_triangle_jumper, B.Cu at (10.2, -115.6)
- added JP33: SolderJumper_2_Open, CUSTOM:small_triangle_jumper, F.Cu at (10.2, -113.0)
- added JP34: SolderJumper_2_Open, CUSTOM:small_triangle_jumper, B.Cu at (10.2, -113.0)
- added JP35: SolderJumper_2_Open, CUSTOM:small_triangle_jumper, F.Cu at (20.3, -128.3)
- added JP36: SolderJumper_2_Open, CUSTOM:small_triangle_jumper, F.Cu at (21.0, -125.7)
- added JP37: SolderJumper_2_Open, CUSTOM:small_triangle_jumper, F.Cu at (20.3, -123.2)
- added JP38: SolderJumper_2_Open, CUSTOM:small_triangle_jumper, F.Cu at (21.0, -121.1)
- added JP39: SolderJumper_2_Open, CUSTOM:small_triangle_jumper, F.Cu at (389.9, 99.1)
- added JP40: SolderJumper_2_Open, CUSTOM:small_triangle_jumper, F.Cu at (390.6, 101.6)
- added JP41: SolderJumper_2_Open, CUSTOM:small_triangle_jumper, F.Cu at (389.9, 104.1)
- added JP42: SolderJumper_2_Open, CUSTOM:small_triangle_jumper, F.Cu at (388.6, 106.7)
- added JP43: SolderJumper_2_Open, CUSTOM:small_triangle_jumper, F.Cu at (387.9, 109.2)
- added JP44: SolderJumper_2_Open, CUSTOM:small_triangle_jumper, F.Cu at (388.6, 111.8)
- added JP45: SolderJumper_2_Open, CUSTOM:small_triangle_jumper, F.Cu at (388.1, 114.3)
- added JP46: SolderJumper_2_Open, CUSTOM:small_triangle_jumper, F.Cu at (388.1, 118.1)
- added JP47: SolderJumper_2_Open, CUSTOM:small_triangle_jumper, F.Cu at (104.1, 304.8)
- added JP48: SolderJumper_2_Open, CUSTOM:small_triangle_jumper, F.Cu at (104.1, 307.3)
- added JP49: SolderJumper_2_Open, CUSTOM:small_triangle_jumper, F.Cu at (104.1, 309.9)
- added JP50: SolderJumper_2_Open, CUSTOM:small_triangle_jumper, F.Cu at (104.1, 312.4)
- added JP51: SolderJumper_2_Open, CUSTOM:small_triangle_jumper, F.Cu at (104.1, 315.0)
- added JP52: SolderJumper_2_Open, CUSTOM:small_triangle_jumper, F.Cu at (104.1, 317.5)
- added JP53: SolderJumper_2_Open, CUSTOM:small_triangle_jumper, F.Cu at (104.1, 320.0)
- added JP54: SolderJumper_2_Open, CUSTOM:small_triangle_jumper, F.Cu at (104.1, 322.6)
- added JP55: SolderJumper_2_Open, CUSTOM:small_triangle_jumper, F.Cu at (407.7, 100.3)
- added JP56: SolderJumper_2_Open, CUSTOM:small_triangle_jumper, F.Cu at (407.7, 102.9)
- added JP57: SolderJumper_2_Open, CUSTOM:small_triangle_jumper, F.Cu at (407.7, 105.4)
- added JP58: SolderJumper_2_Open, CUSTOM:small_triangle_jumper, F.Cu at (125.7, 303.5)
- added JP59: SolderJumper_2_Open, CUSTOM:small_triangle_jumper, F.Cu at (125.7, 306.1)
- added JP60: SolderJumper_2_Open, CUSTOM:small_triangle_jumper, F.Cu at (125.7, 308.6)
- added JP61: SolderJumper_2_Open, CUSTOM:small_triangle_jumper, F.Cu at (405.7, 109.2)
- added JP62: SolderJumper_2_Open, CUSTOM:small_triangle_jumper, F.Cu at (405.7, 111.8)
- added JP63: SolderJumper_2_Open, CUSTOM:small_triangle_jumper, F.Cu at (405.7, 114.3)
- added JP64: SolderJumper_2_Open, CUSTOM:small_triangle_jumper, F.Cu at (405.7, 116.8)
- added JP65: SolderJumper_2_Open, CUSTOM:small_triangle_jumper, F.Cu at (126.3, 315.0)
- added JP66: SolderJumper_2_Open, CUSTOM:small_triangle_jumper, F.Cu at (126.3, 317.5)
- added JP67: SolderJumper_2_Open, CUSTOM:small_triangle_jumper, F.Cu at (126.5, 320.0)
- added JP68: SolderJumper_2_Open, CUSTOM:small_triangle_jumper, F.Cu at (127.0, 322.6)
- added JP69: SolderJumper_2_Open, CUSTOM:small_triangle_jumper, F.Cu at (415.3, 109.2)
- added JP70: SolderJumper_2_Open, CUSTOM:small_triangle_jumper, F.Cu at (136.4, 303.5)
- added JP71: SolderJumper_2_Open, CUSTOM:small_triangle_jumper, F.Cu at (415.3, 111.8)
- added JP72: SolderJumper_2_Open, CUSTOM:small_triangle_jumper, F.Cu at (137.2, 306.1)
- added JP73: SolderJumper_2_Open, CUSTOM:small_triangle_jumper, F.Cu at (415.3, 114.3)
- added JP74: SolderJumper_2_Open, CUSTOM:small_triangle_jumper, F.Cu at (415.3, 116.8)
- added JP75: SolderJumper_2_Open, CUSTOM:small_triangle_jumper, F.Cu at (135.9, 311.1)
- added JP76: SolderJumper_2_Open, CUSTOM:small_triangle_jumper, F.Cu at (135.9, 313.7)
- added TP5: ATM_SPARE, TestPoint:TestPoint_Pad_D1.0mm, F.Cu at (244.8, 19.1)
- C16, C19, C33, C36, C50, C53, C67, C70: footprint Capacitor_SMD:C_0603_1608Metric -> Capacitor_SMD:C_0603_1608Metric_Pad1.05x0.95mm_HandSolder
- C21, C22, C24, C47, C48, C49, JP10, JP13, JP15, JP2, JP4, JP6, JP8, Q5, Q6, R114, R117, R118, R122, R123: moved to B.Cu
- Y1: footprint Crystal:Crystal_SMD_HC49-SD_HandSoldering -> CUSTOM:CX5032GB10000H0PESZZ
- moved R113 386.0 mm to (-30.5, -109.2)
- moved R112 375.4 mm to (-30.5, -106.7)
- moved R110 373.5 mm to (-17.8, -102.9), turned to 90 degrees
- moved R111 369.8 mm to (-20.3, -102.9), turned to 90 degrees
- moved C44 369.4 mm to (-20.3, -109.2), turned to 270 degrees
- moved Q5 368.3 mm to (-19.1, -109.2), turned to 90 degrees
- moved C45 367.4 mm to (-14.0, -109.2), turned to 270 degrees
- moved C46 365.6 mm to (-16.5, -109.2), turned to 270 degrees
- moved R114 364.4 mm to (-25.4, -108.0), turned to 270 degrees
- moved C34 363.8 mm to (-75.2, -90.9)
- moved C35 363.8 mm to (-70.9, -88.4)
- moved C36 363.8 mm to (-53.3, -94.1)
- moved C37 363.8 mm to (-73.7, -99.7)
- moved C38 363.8 mm to (-80.4, -90.0)
- moved C39 363.8 mm to (-62.3, -93.2)
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Connections:
- J10 pad 4: /DRIVE_1/ENC_B -> /DRIVE_1/ENC_A
- J10 pad 5: /DRIVE_1/ENC_A -> /DRIVE_1/ENC_B
Other:
- board size 100 x 100 mm -> 200 x 100 mm
